Commit message: change path for meshes

File: urdf/r24_description.urdf (robot description, URDF)
Before this commit: robot r24_description, 9 links, 8 joints
Links:
- link back_left_link: geometry collision mesh filename=package://meshes/back_left_link.STL; visual mesh filename=package://meshes/back_left_link.STL
- link back_right_link: geometry collision mesh filename=package://meshes/back_right_link.STL; visual mesh filename=package://meshes/back_right_link.STL
- link base_link: geometry collision mesh filename=package://meshes/base_link.STL; visual mesh filename=package://meshes/base_link.STL
- link camera_link: geometry collision mesh filename=package://meshes/stereocam_link.STL; visual mesh filename=package://r24_description/meshes/stereocam_link.STL
- link front_left_link: geometry collision mesh filename=package://meshes/front_left_link.STL; visual mesh filename=package://meshes/front_left_link.STL
- link front_right_link: geometry collision mesh filename=package://meshes/front_right_link.STL; visual mesh filename=package://meshes/front_right_link.STL
